File: PCB/ESP32SATTRACKER.kicad_sch (KiCad schematic)
At the start: 10 parts, among them J1 Conn_01x19_Socket, J2 Conn_01x19_Socket, U1 LM2596S-5, U3 74HCT244

Commit message: 80% completed
Parts:
- added C1, C2: 100uF, symbol Device:C_Polarized
- added J3, J4: Screw_Terminal_01x04, TerminalBlock_4Ucon:TerminalBlock_4Ucon_1x04_P3.50mm_Horizontal, symbol Connector:Screw_Terminal_01x04
- A1: value Pololu_Breakout_A4988 -> A4988 X-AXIS
- A2: value Pololu_Breakout_A4988 -> A4988 Y-AXIS
Connections:
- net +5V: now also A1.10 (MS1), A1.11 (MS2), A1.12 (MS3), A1.2 (VDD), A2.10 (MS1), A2.11 (MS2), A2.12 (MS3), A2.2 (VDD), U3.20 (VCC)
- net GND: now also A1.1 (GND), A1.7 (GND), A2.1 (GND), A2.7 (GND), C1.2, C2.2
- net P25: now also A1.9 (~{ENABLE}), A2.9 (~{ENABLE})
- net VBUS: now also A1.8 (VMOT), A2.8 (VMOT), C1.1, C2.1
- net at A2.13 (~{RESET}): now also A2.14 (~{SLEEP})
- net at A2.3 (1B): now also J4.1 (Pin_1)
- net at A2.4 (1A): now also J4.2 (Pin_2)
- net at A2.5 (2A): now also J4.3 (Pin_3)
- net at A2.6 (2B): now also J4.4 (Pin_4)
- net at A1.13 (~{RESET}): now also A1.14 (~{SLEEP})
- net at A1.3 (1B): now also J3.1 (Pin_1)
- net at A1.4 (1A): now also J3.2 (Pin_2)
- net at A1.5 (2A): now also J3.3 (Pin_3)
- net at A1.6 (2B): now also J3.4 (Pin_4)
Other:
- moved on the sheet: A1, A2, J1, J2, U3

Commit message: completed diagram
Parts:
- added J5: Conn_01x14_Socket, symbol Connector:Conn_01x14_Socket
- added J6: Conn_01x04_Socket, symbol Connector:Conn_01x04_Socket
- added J7: Screw_Terminal_01x02, TerminalBlock_4Ucon:TerminalBlock_4Ucon_1x02_P3.50mm_Vertical, symbol Connector:Screw_Terminal_01x02
- added J8: Conn_01x05_Socket, symbol Connector:Conn_01x05_Socket
Connections:
- net GND: now also U3.1 (1OE), U3.10 (GND), U3.19 (2OE), J5.13 (Pin_13), J7.1 (Pin_1), J8.1 (Pin_1), J8.4 (Pin_4)
- net P14: now also U3.4 (1A1)
- net P15: now also J5.12 (Pin_12)
- net P18: now also J5.8 (Pin_8), J6.1 (Pin_1)
- net P19: now also J6.2 (Pin_2)
- net P2: now also J5.10 (Pin_10)
- net P21: now also J8.2 (Pin_2)
- net P22: now also J8.3 (Pin_3)
- net P23: now also J5.9 (Pin_9), J6.3 (Pin_3)
- net P26: now also U3.8 (1A3)
- net P27: now also U3.6 (1A2)
- net P32: now also U3.2 (1A0), J6.4 (Pin_4)
- net P5: now also J5.11 (Pin_11)
- net VBUS: now also J7.2 (Pin_2)
- net Y2: now reaches A2.15 (STEP)
- net Y2: now also U3.14 (1Y2)
- net Y3: now reaches A2.16 (DIR)
- net Y3: now also U3.12 (1Y3)
- net Y1: now reaches U3.16 (1Y1)
- net Y1: now also A1.16 (DIR)
- net Y0: now reaches U3.18 (1Y0)
- net Y0: now also A1.15 (STEP)
- new net +3V3: J5.14 (Pin_14), J5.7 (Pin_7), J8.5 (Pin_5)
- no-connect marks 0 -> 14
Other:
- note added: "CS"
- note added: "DC"
- note added: "GND"
- note added: "LED"
- note added: "RST"
- note added: "SCK"
- note added: "SDI(MOSI)"
- note added: "SD_CS"
- note added: "SD_MISO"
- note added: "SD_MOSI"
- note added: "SD_SCK"
- note added: "VCC"
- moved on the sheet: U3

Commit message: assigned footprints
Parts:
- 220uF1: renamed from 220uF; footprint (none) -> Capacitor_THT:CP_Radial_D8.0mm_P3.50mm
- 680uF1: renamed from 680uF; footprint (none) -> Capacitor_THT:CP_Radial_D10.0mm_P5.00mm
- C1, C2: footprint (none) -> Capacitor_THT:CP_Radial_D8.0mm_P3.50mm
- D1: footprint (none) -> Diode_THT:D_DO-201AD_P15.24mm_Horizontal
- J5: footprint (none) -> Connector_PinHeader_2.54mm:PinHeader_1x14_P2.54mm_Vertical
- J6: footprint (none) -> Connector_PinHeader_2.54mm:PinHeader_1x04_P2.54mm_Vertical
- J8: footprint (none) -> Connector_PinHeader_2.54mm:PinHeader_1x05_P2.54mm_Vertical
- L1: footprint (none) -> Inductor_SMD:L_12x12mm_H8mm
- U3: footprint (none) -> Package_DIP:DIP-20_W7.62mm
Changed lines of the file:
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@@
 		(on_board yes)
 		(dnp no)
-		(property "Reference" "220uF"
+		(property "Reference" "220uF1"
 			(at 122.936 174.498 0)
 			(effects
@@
 			)
 		)
-		(property "Footprint" ""
+		(property "Footprint" "Capacitor_THT:CP_Radial_D8.0mm_P3.50mm"
 			(at 120.3452 177.8 0)
 			(effects
@@
 			(project "ESP32SATTRACKER"
 				(path "/32988a15-4770-44e4-947e-567ab63aff84"
-					(reference "220uF")
+					(reference "220uF1")
 					(unit 1)
 				)
@@
 			)
 		)
-		(property "Footprint" ""
+		(property "Footprint" "Capacitor_THT:CP_Radial_D8.0mm_P3.50mm"
 			(at 198.12 94.2848 0)
 			(effects
@@
 		(on_board yes)
 		(dnp no)
-		(property "Reference" "680uF"
+		(property "Reference" "680uF1"
 			(at 50.546 173.228 0)
 			(effects
@@
 			)
 		)
-		(property "Footprint" ""
+		(property "Footprint" "Capacitor_THT:CP_Radial_D10.0mm_P5.00mm"
 			(at 47.9552 176.53 0)
 			(effects
@@
 			(project ""
 				(path "/32988a15-4770-44e4-947e-567ab63aff84"
-					(reference "680uF")
+					(reference "680uF1")
 					(unit 1)
 				)
@@
 			)
 		)
-		(property "Footprint" ""
+		(property "Footprint" "Connector_PinHeader_2.54mm:PinHeader_1x04_P2.54mm_Vertical"
 			(at 132.08 24.13 0)
 			(effects
@@
 			)
 		)
-		(property "Footprint" ""
+		(property "Footprint" "Inductor_SMD:L_12x12mm_H8mm"
 			(at 107.95 170.18 0)
 			(effects
@@
 			)
 		)
-		(property "Footprint" ""
+		(property "Footprint" "Diode_THT:D_DO-201AD_P15.24mm_Horizontal"
 			(at 92.71 173.99 0)
 			(effects
@@
 			)
 		)
-		(property "Footprint" ""
+		(property "Footprint" "Connector_PinHeader_2.54mm:PinHeader_1x05_P2.54mm_Vertical"
 			(at 87.63 124.46 0)
 			(effects
@@
 			)
 		)
-		(property "Footprint" ""
+		(property "Footprint" "Connector_PinHeader_2.54mm:PinHeader_1x14_P2.54mm_Vertical"
 			(at 133.35 55.88 0)
 			(effects
@@
 			)
 		)
-		(property "Footprint" ""
+		(property "Footprint" "Capacitor_THT:CP_Radial_D8.0mm_P3.50mm"
 			(at 267.97 93.0148 0)
 			(effects
@@
 			)
 		)
-		(property "Footprint" ""
+		(property "Footprint" "Package_DIP:DIP-20_W7.62mm"
 			(at 208.28 46.99 0)
 			(effects

Commit message: completed the PCB
Parts:
- 220uF1, C1, C2: footprint Capacitor_THT:CP_Radial_D8.0mm_P3.50mm -> Capacitor_THT:CP_Axial_L11.0mm_D6.0mm_P18.00mm_Horizontal
- 680uF1: footprint Capacitor_THT:CP_Radial_D10.0mm_P5.00mm -> Capacitor_THT:CP_Axial_L18.0mm_D10.0mm_P25.00mm_Horizontal
Changed lines of the file:
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@@
 			)
 		)
-		(property "Footprint" "Capacitor_THT:CP_Radial_D8.0mm_P3.50mm"
+		(property "Footprint" "Capacitor_THT:CP_Axial_L11.0mm_D6.0mm_P18.00mm_Horizontal"
 			(at 120.3452 177.8 0)
 			(effects
@@
 			)
 		)
-		(property "Footprint" "Capacitor_THT:CP_Radial_D8.0mm_P3.50mm"
+		(property "Footprint" "Capacitor_THT:CP_Axial_L11.0mm_D6.0mm_P18.00mm_Horizontal"
 			(at 198.12 94.2848 0)
 			(effects
@@
 			)
 		)
-		(property "Footprint" "Capacitor_THT:CP_Radial_D10.0mm_P5.00mm"
+		(property "Footprint" "Capacitor_THT:CP_Axial_L18.0mm_D10.0mm_P25.00mm_Horizontal"
 			(at 47.9552 176.53 0)
 			(effects
@@
 			)
 		)
-		(property "Footprint" "Capacitor_THT:CP_Radial_D8.0mm_P3.50mm"
+		(property "Footprint" "Capacitor_THT:CP_Axial_L11.0mm_D6.0mm_P18.00mm_Horizontal"
 			(at 267.97 93.0148 0)
 			(effects

Commit message: Update README with open source badges and PCB placeholder
Parts:
- added H1, H2, H3, H4, H5: MountingHole_Pad, MountingHole:MountingHole_2.2mm_M2_Pad, symbol Mechanical:MountingHole_Pad
Connections:
- net 3V3 is gone; now on net +3V3: J1.19 (Pin_19)
- net GND: now also H1.1, H2.1, H3.1, H4.1, H5.1
