File: PCB/ESP32SATTRACKER.kicad_pcb (KiCad board)
At the start: 2 copper layers, 132.2 x 137 mm, 18 parts, among them J1 Conn_01x19_Socket, J2 Conn_01x19_Socket, J3 Screw_Terminal_01x04, J4 Screw_Terminal_01x04, J5 Conn_01x14_Socket, J6 Conn_01x04_Socket, J7 Screw_Terminal_01x02, J8 Conn_01x05_Socket, U1 LM2596S-5, U3 74HCT244

Commit message: Update README with open source badges and PCB placeholder
Parts:
- added G***: LOGO, PCB:REPOQR, B.Cu at (112.2, 129.6)
- added G***: LOGO, PCB:NSQR, B.Cu at (172.3, 61.9)
- added H1: MountingHole_Pad, MountingHole:MountingHole_2.2mm_M2_Pad, F.Cu at (81.6, 161.4)
- added H2: MountingHole_Pad, MountingHole:MountingHole_2.2mm_M2_Pad, F.Cu at (197.7, 37.8)
- added H3: MountingHole_Pad, MountingHole:MountingHole_2.2mm_M2_Pad, F.Cu at (77.5, 37.3)
- added H4: MountingHole_Pad, MountingHole:MountingHole_2.2mm_M2_Pad, F.Cu at (199.4, 130.0)
- added H5: MountingHole_Pad, MountingHole:MountingHole_2.2mm_M2_Pad, F.Cu at (139.2, 129.5)
- moved J5 33.0 mm to (93.8, 89.7), turned to 90 degrees
- moved J6 7.60 mm to (106.7, 162.1), turned to 90 degrees
Connections:
- J1 pad 19: /3V3 -> +3V3
Routing:
- net +5V: track 128.0 -> 202.3 mm, vias 0 -> 2
- net +3V3: track 24.8 -> 64.0 mm, vias 2 -> 5
- net /P15: track 40.3 -> 15.5 mm
- net /P18: track 88.1 -> 103.0 mm
- net /P23: track 94.6 -> 105.7 mm
- net /P19: track 98.2 -> 87.9 mm
- net GND: track 0.00 -> 10.1 mm, vias 11 -> 399
- net /P2: track 25.7 -> 16.5 mm
- net /P32: track 156.8 -> 150.5 mm
- net Net-(A1-~{RESET}): track 0.00 -> 2.54 mm
- net unconnected-(J5-Pin_3-Pad3): track 0.00 -> 1.77 mm
- net VBUS: track 209.4 -> 210.3 mm
- net /P5: track 17.5 -> 16.7 mm
- net unconnected-(J5-Pin_6-Pad6): vias 0 -> 1
- net unconnected-(J5-Pin_4-Pad4): vias 0 -> 1
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- added copper zone on F.Cu, net (none)
Other:
- board text added: "+"
- board text added: "-"
- board text added: "12V INPUT"
- board text added: "1A"
- board text added: "1B"
- board text added: "2.4{dblquote} TFT SCREEN"
- board text added: "2A"
- board text added: "2B"
- board text added: "5A MAX"
- board text added: "AD0"
- board text added: "CS"
- board text added: "DC"
- board text added: "DESIGNED IN PAKISTAN"
- board text added: "Designed by Muhammad Uzzam Butt"
- board text added: "ESP-32 SATTELITE TRACKING COMPUTER"
- board text added: "ESP32-S"
- board text added: "GND"
- board text added: "LED"
- board text added: "NORTHERNSTUDIOS.CC"
- board text added: "RST"
- board text added: "SCK"
- board text added: "SCL"
- board text added: "SDA"
- board text added: "SDI(MOSI)"
- board text added: "SD_CS"
- board text added: "SD_MISO"
- board text added: "SD_MOSI"
- board text added: "STEP_AZI"
- board text added: "STEP_ELE"
- board text added: "VCC"
- board text added: "{ "ViaStitching": "0.2", "stitch_zone_0": { "HSpacing": "3", "VSpacing": "3", "HOffset": "0", "VOffset": "0", "Clearance": "0", "Randomize": false } }"
- board text added: "{ "ViaStitching": "0.2", "stitch_zone_0": { "HSpacing": "5", "VSpacing": "5", "HOffset": "0", "VOffset": "0", "Clearance": "0.2", "Randomize": false } }"

Commit message: rerouted the ESP32, IMU AND TFT AGAIN CUZ I AGAIN MESSED UP THE ESP32 ARRANGEMENT AND INVERTED IT!!
Parts:
- removed the G*** at (172.3, 61.9)
- added G***: LOGO, LOGO, B.Cu at (190.1, 85.0)
- moved J1 20.2 mm to (134.2, 76.3)
- moved J2 20.1 mm to (134.3, 56.2)
- moved G*** 2.28 mm to (110.0, 130.2)
Routing:
- net /P2: track 16.5 -> 43.0 mm
- net +3V3: track 64.0 -> 38.3 mm, vias 5 -> 3
- net /P15: track 15.5 -> 36.8 mm
- net /P14: track 17.0 -> 37.4 mm
- net /P27: track 17.3 -> 37.4 mm
- net /P26: track 18.3 -> 38.4 mm
- net /P5: track 16.7 -> 36.7 mm
- net /P19: track 87.9 -> 107.2 mm
- net /P23: track 105.7 -> 119.9 mm
- net +5V: track 202.3 -> 216.1 mm
- net /P18: track 103.0 -> 111.9 mm
- net /P21: track 28.1 -> 36.4 mm
- net GND: track 10.1 -> 5.08 mm, vias 399 -> 400
- net /P32: track 150.5 -> 146.5 mm
- net /P25: track 118.5 -> 116.1 mm
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